File: v2/Power_amplifier.kicad_sch (KiCad schematic)
At the start: 44 parts, among them U18 TPA3132D2RHBR

Commit message: Most v2 changes made
Parts:
- removed C105, C116, C117: 1n, Capacitor_SMD:C_0603_1608Metric_Pad1.08x0.95mm_HandSolder, symbol UAM_symbols:C
- removed C76, C93: 1n,50V, Capacitor_SMD:C_0603_1608Metric_Pad1.08x0.95mm_HandSolder, symbol UAM_symbols:C
- removed C77, C89: 100n,50V, Capacitor_SMD:C_0603_1608Metric_Pad1.08x0.95mm_HandSolder, symbol UAM_symbols:C
- removed C78, C86: 220u, Capacitor_THT:CP_Radial_D10.0mm_P5.00mm, symbol UAM_symbols:C_Polarized_US
- removed C79, C81, C85, C88: 1u, Capacitor_SMD:C_0603_1608Metric_Pad1.08x0.95mm_HandSolder, symbol UAM_symbols:C
- removed C80, C87, C92, C95: 220n,50V, Capacitor_SMD:C_0603_1608Metric_Pad1.08x0.95mm_HandSolder, symbol UAM_symbols:C
- removed JP3, JP4, JP5: SolderJumper_2_Open, Jumper:SolderJumper-2_P1.3mm_Open_RoundedPad1.0x1.5mm, symbol UAM_symbols:SolderJumper_2_Open
- removed L3, L4: 22u, Inductor:SPM7054VC, symbol Device:L
- removed R44: 5k6, Resistor_SMD:R_0603_1608Metric_Pad0.98x0.95mm_HandSolder, symbol UAM_symbols:R_US
- removed R45: ~, Resistor_SMD:R_0603_1608Metric_Pad0.98x0.95mm_HandSolder, symbol UAM_symbols:R_US
- removed R46, R49, R50, R52: 100k, Resistor_SMD:R_0603_1608Metric_Pad0.98x0.95mm_HandSolder, symbol UAM_symbols:R_US
- removed R47: 56k, Resistor_SMD:R_0603_1608Metric_Pad0.98x0.95mm_HandSolder, symbol UAM_symbols:R_US
- removed R48: 36k, Resistor_SMD:R_0603_1608Metric_Pad0.98x0.95mm_HandSolder, symbol UAM_symbols:R_US
- removed R51: 330R, Resistor_SMD:R_0603_1608Metric_Pad0.98x0.95mm_HandSolder, symbol UAM_symbols:R_US
- removed R54: 10k, Resistor_SMD:R_0603_1608Metric_Pad0.98x0.95mm_HandSolder, symbol UAM_symbols:R_US
- removed U18: TPA3132D2RHBR, Package_DFN_QFN:VQFN-32-1EP_5x5mm_P0.5mm_EP3.5x3.5mm, symbol UAM_symbols:TPA3132D2RHBR
- added C55, C59: 100p, symbol Device:C_Small
- added C56, C57: 100n, symbol Device:C_Small
- added C58: 121p, symbol Device:C_Small
- added C60: 715p, symbol Device:C_Small
- added C61, C63, C67, C69, C70, C71, C72, C73: 1u, symbol Device:C
- added C62, C65, C75: 330u, symbol Device:C_Polarized_US
- added C64, C66, C68: 100n, symbol Device:C
- added C74: 10n, symbol Device:C_Small
- added C76, C77, C79, C80: 33n, symbol Device:C_Small
- added C78: 0u1, symbol Device:C
- added L3, L4: 22u, NRS6045T100MMGK:IND_TAIYO_NRS6045_TAY, symbol UAM_symbols:L_Ferrite
- added Q4: DMP6050SSD, Package_SO:SOIC-8_3.9x4.9mm_P1.27mm, symbol Transistor_FET:DMP6050SSD
- added Q5, Q6, Q7: TBC847B,LM, UAM_footprints:TBC847BLM, symbol UAM_symbols:TBC847B,LM
- added R35: 12k1, symbol Device:R_US
- added R36: 17k4, symbol Device:R_US
- added R37, R38, R44, R45, R46, R47: 100k, symbol Device:R_US
- added R39, R40: 100, symbol Device:R_US
- added R41, R42: 10k, symbol Device:R_US
- added R43: 4k75, symbol Device:R_US
- added R48: 7k5, symbol Device:R_US
- added R49, R50: 3R3, symbol Device:R_Small_US
- added R51: 22k, symbol Device:R_US
- added R52: 30k,1%, symbol Device:R_US
- added TP15: TestPoint, symbol UAM_symbols:TestPoint
- added U10, U11: OPA1677DBVR, UAM_footprints:SOT23_DBV0005A_TEX, symbol UAM_symbols:OPA1677DBVR
- added U12: TPA3244DDWR, UAM_footprints:TPA3244DDW, symbol UAM_symbols:TPA3244DDWR
- added Z1, Z2, Z3: BZT52C15-7-F, UAM_footprints:SOD3716X145N, symbol UAM_symbols:BZT52C15-7-F
- C81: renamed from C91; value 1u,50V -> 220n,100V
- C82: renamed from C83; value 1u,50V -> 220n,100V
- TP16: footprint TestPoint:TestPoint_Pad_D1.0mm -> (none)
- renumbered C94 to C83, C82 to C84, C90 to C85, C84 to C86, R55 to R53, R53 to R54, TP15 to TP18
Connections:
- net DAC_TRANSDUCER is gone; now on net AMP_L: TP16.1
- net AMP_L: now also L4.2
- net AMP_R: now also L3.2, TP15.1
- net GND: now also C55.2, C59.1, C62.2, C64.1, C66.1, C68.1, C71.1, C72.1, C73.2, C74.1, C78.2, Q5.2 (E), Q6.2 (E), R44.2, R45.2, R46.2, R47.2, R51.1, R52.1, U12.10 (GND), U12.11 (GND), U12.20 (M1), U12.25 (GND), U12.26 (GND), U12.33 (GND), U12.34 (GND), U12.41 (GND), U12.42 (GND), U12.45 (PowerPAD), U12.6 (INPUT_D), U12.7 (INPUT_C)
- net OUT_L: now also C77.2, C80.2, L4.1, U12.32 (OUT_B), U12.39 (OUT_D), U12.40 (OUT_D)
- net OUT_R: now also C76.2, C79.2, L3.1, U12.27 (OUT_A), U12.28 (OUT_A), U12.35 (OUT_C)
- new net: R51.2, U12.16 (OC_ADJ)
- new net: C60.1, C67.1, U11.1 (OUT), U11.4 (-)
- new net: C67.2, U12.18 (INPUT_A)
- new net: C56.2, Q5.3 (C), R37.2, R39.2
- new net: C72.2, U12.17 (INPUT_B)
- new net: C58.1, R35.2, R36.1
- new net: C58.2, R43.1, U10.1 (OUT), U10.4 (-)
- new net: R38.1, Z2.2 (A)
- new net: Q6.1 (B), R42.1, R45.1
- new net: C60.2, R43.2, R48.1
- new net: C59.2, R48.2, U11.3 (+)
- new net: C73.1, U12.9 (AVDD)
- new net: C61.1, C63.1, C65.1, C69.1, C70.1, C75.1, Q4.7 (D1), Q4.8 (D1), R46.1, U12.29 (PVDD_AB), U12.30 (PVDD_AB), U12.31 (PVDD_AB), U12.36 (PVDD_CD), U12.37 (PVDD_CD), U12.38 (PVDD_CD)
- new net: C61.2, C63.2, C65.2
- new net: C62.1, C64.2, Q4.5 (D2), Q4.6 (D2), R47.1, R49.2, R50.2, U12.21 (VDD)
- new net: C55.1, R36.2, U10.3 (+)
- new net: C69.2, C70.2, C75.2
- new net: C80.1, U12.24 (BST_B)
- new net: Q5.1 (B), R41.1, R44.1
- new net: C68.2, R50.1, U12.1 (GVDD_CD)
- new net: R52.2, U12.15 (FREQ_ADJ)
- new net: C66.2, R49.1, U12.22 (GVDD_AB)
- new net: C76.1, U12.23 (BST_A)
- new net: C78.1, U12.3 (VBG)
- new net: C79.1, U12.43 (BST_C)
- new net: C77.1, U12.44 (BST_D)
- new net: C74.2, U12.8 (C_START)
- new net: Q4.4 (G2), R40.1
- new net: C57.2, Q6.3 (C), R38.2, R40.2
- new net: R37.1, Z1.2 (A)
- new net: Q4.2 (G1), R39.1
- new net +12V: C57.1, Q4.3 (S2), Z2.1 (K)
- new net +3.3V: U10.5 (V+), U11.5 (V+)
- new net +30V: C56.1, Q4.1 (S1), Z1.1 (K)
- new net -3V3: U10.2 (V-), U11.2 (V-)
- new net AMP_Pwr_Switch: R41.2, R42.2
- new net DAC_TO_PAMP: R35.1
- new net DVDD: C71.2, U12.12 (DVDD), U12.19 (M2)
- new net TPA_CLIP_OTW: U12.2 (CLIP_OTW_N)
- new net TPA_FAULT: U12.4 (FAULT_N)
- new net TPA_RESET: U12.5 (RESET_N)
- no-connect marks 1 -> 2
Other:
- note added: "1uF decoupling caps should be placed as close as possible to PVDD pins"
- note added: "4th Order Butterworth Lowpass Filter Passband = 100kHz See: DAC_to_AMP_LPF_Design_Report.pdf *At end of design, see if similar C/R values already exist to save cost/complexity."
- note added: "At 155C, device enters thermal shutdown and device must be reset to resume normal operation."
- note added: "Datasheet recommends 470uF electrolytic caps for decoupling, but since we are not operating at max power, 330u is sufficient"
- note added: "FAULT and CLIP_OTW have internal pullups to 3.3V"
- note added: "FREQ_ADJ determines frame rate for AM interference avoidance. Currently set for nominal and master mode"
- note added: "High Side Simultaneous Power Switching STM32 needs to output HIGH for TPA3244 to be powered. *If layout is difficult, dual channel PMOS can be changed to two single PMOS"
- note added: "M2 M1 = 1 0 for PBTL"
- note added: "OC_ADJ resistor sets protection mode (CB3C or Latched OC) and OC threshold, between 22k and 64k."
- note added: "RC Snubber"
- note added: "RC filters separate VDD and GVDD, as recommended in datasheet."
- note added: "Recommended to monitor CLIP_OTW and respond to OTE by turning down volume to prevent overheating of device."
- note added: "Recommended to release RESET after power supply is settled for minimum turn on audible artefacts. Note: Asserting RESET low initiates device ramp down and forces FAULT high. For thermal reliability, rising edge of RESET must occur no sooner than 4ms after falling edge of FAULT."
- note added: "Using same RC snubber as before, may need tweaking"
- note removed: "GAIN CONTROL"
- note removed: "R-C Snubber"
- note removed: "RC filter with cutoff-frequency 106 kHz. Output impedance of DAC with buffer: 1k5"
- note removed: "Tolerance of these components does not significantly impact power factor"
- company: Power Amplifier -> (none)
- title: RM -> (none)
- moved on the sheet: C81, C82, C83, C84, C85, C86, R53, R54, TP17, TP18
