File: v2/src/BPF.kicad_sch (KiCad schematic)
At the start: 24 parts, among them U25 LMV641MFX/NOPB, U26 LMV641MFX/NOPB, U27 LMV641MFX/NOPB

Commit message: v2.0 final version including minor hardware revisions
Parts:
- R108: renamed from R120; LCSC PN C22763 -> C858885
- renumbered C129 to C128, C130 to C129, C131 to C130, C132 to C131, C133 to C132, C134 to C133, C135 to C134, C136 to C135, C137 to C136, C138 to C137, C139 to C138, C140 to C139, R113 to R101, R114 to R102, R115 to R103, R116 to R104, R117 to R105, R118 to R106, R119 to R107, R121 to R109, U25 to U28, U26 to U29, U27 to U30
Connections:
- net GND: now also U28.3 (+), U29.3 (+), U30.3 (+); no longer U28.4 (-), U29.4 (-), U30.4 (-)
- net at C138.2, R109.2: now also U30.4 (-); no longer U30.3 (+)
- net at C136.2, R106.2: now also U29.4 (-); no longer U29.3 (+)
- net at C132.2, R103.2: now also U28.4 (-); no longer U28.3 (+)
- net PREAMP_LPF renamed PREAMP_BPF
