File: v2/src/Board_Management.kicad_sch (KiCad schematic)
At the start: 28 parts, among them Q12 BSS138, Q13 BSS138, Q14 BSS138, Q15 BSS138, U18 LPS22HH, U19 INA219AIDCNR

Commit message: v2.0 final version including minor hardware revisions
Parts:
- added R116: 100k, Resistor_SMD:R_0603_1608Metric, symbol UAM_symbols:R_US
- renumbered C106 to C104, C107 to C106, Q12 to Q6, Q13 to Q7, Q14 to Q8, Q15 to Q9, R78 to R66, R79 to R67, R80 to R68, R81 to R69, R82 to R70, R83 to R71, R84 to R72, R85 to R73, R86 to R74, R87 to R75, R88 to R76, R89 to R77, R90 to R78, R91 to R79, R92 to R80, U18 to U21, U19 to U22
Connections:
- net +3V3: now also R116.1
- net PRESS_CS#: now also R116.2
Other:
- moved on the sheet: C104, U21
