File: v2/src/Connections.kicad_sch (KiCad schematic)
At the start: 40 parts, among them J3 USB_B_Micro, J5 2601-1102, J6 2601-1103, Q8 GSFD6959, U13 TPD4E05U06DQA, U14 USB3343, U15 TPD4E05U06DQA, Y3 26 MHz

Commit message: v2.0 final version including minor hardware revisions
Parts:
- removed Q8: GSFD6959, OpenAquatix-Hardware_footprints:PMOSGDS_TO-252_DPAK_GAS, symbol UAM_symbols:GSFD6959
- removed R51, R52, R53, R54, R55, R56, R57, R58: 22R, Resistor_SMD:R_0603_1608Metric, symbol Device:R_US
- removed R59, R60: 0R, Resistor_SMD:R_0603_1608Metric, symbol Device:R_US
- removed R61: 100k, Resistor_SMD:R_0603_1608Metric, symbol Device:R_US
- added Q3: Si7617DN, Package_SO:Vishay_PowerPAK_1212-8_Single, symbol Transistor_FET:Si7617DN
- added R49: 1M, Resistor_SMD:R_0603_1608Metric, symbol UAM_symbols:R_US
- renumbered C63 to C62, C64 to C63, C65 to C64, C66 to C65, C67 to C66, C68 to C67, C69 to C68, R42 to R40, R43 to R41, R46 to R42, R47 to R43, R48 to R44, R49 to R45, R44 to R46, R45 to R47, R50 to R48, U13 to U16, U14 to U17, U15 to U18
Connections:
- net +3.3V is gone; now on net +3V3: C68.1, J4.4 (3V3), U17.9 (VDDIO)
- net +BATTa: now also Q3.1 (S), Q3.2 (S), Q3.3 (S)
- net GND: now also J5.3 (2_1), J5.4 (2_2), R49.1; no longer J5.1 (1_1), J5.2 (1_2)
- net ULPI_D0: now also U17.4 (DATA0)
- net ULPI_D1: now also U17.5 (DATA1)
- net ULPI_D2: now also U17.6 (DATA2)
- net ULPI_D3: now also U17.7 (DATA3)
- net ULPI_D4: now also U17.8 (DATA4)
- net ULPI_D5: now also U17.10 (DATA5)
- net ULPI_D6: now also U17.11 (DATA6)
- net ULPI_D7: now also U17.12 (DATA7)
- net ULPI_DIR: now also U17.1 (DIR)
- net ULPI_NXT: now also U17.3 (NXT)
- net at D4.2 (A): now also Q3.4 (G), R49.2
- net PWR_IN2: now reaches D3.1 (A1), F1.2
- net PWR_IN2: now also Q3.5 (D)
- net +3V3: now reaches C65.2, U17.16 (VBAT)
- new net PWR_IN1: F1.1, J5.1 (1_1), J5.2 (1_2)
Other:
- note added: "Clamp V_GS to 12V in case V_in > 25V"
- note added: "P-Channel MOSFET for RPP: R_DS(on) = 12mOhm V_DS(max) = -30V V_GS(max) = +/- 25V"
- note added: "Place CLK resistor near PHY"
- note added: "Typical hydrophone connections have shield, negative, and positive. Positive between shield and negative for additional shielding"
- note removed: "Clamp V_GS to 12V in case V_in > 20V"
- note removed: "P-Channel MOSFET for RPP: R_DS(on) = 12mOhm V_DS(max) = -60V V_GS(max) = +/- 20V"
- note removed: "Place CLK, DIR, NXT resistors near PHY Place DATA, STP resistors near uC"
- moved on the sheet: F1, J5
