File: v2/src/DC-DC.kicad_sch (KiCad schematic)
At the start: 78 parts, among them Q4 DMP3068L-7, Q5 BSS138, Q6 BSS138, Q7 CSD18543Q3A, SW3 CS12ANW03, U10 TLV75733PDYDR, U11 TLV75733PDYDR, U12 LMR54406, U6 LMQ66430R5RXBR, U7 TPS60403DBV, U8 LM5155DSSR, U9 TPS72301DBV

Commit message: v2.0 final version including minor hardware revisions
Parts:
- removed C28: 4u7,50V, Capacitor_SMD:C_1210_3225Metric, symbol UAM_symbols:C
- removed Q4: DMP3068L-7, Package_TO_SOT_SMD:SOT-23, symbol Transistor_FET:DMP3099L
- removed Q5, Q6: BSS138, Package_TO_SOT_SMD:SOT-23, symbol UAM_symbols:BSS138
- removed R24: 2k, Resistor_SMD:R_0603_1608Metric, symbol Device:R_US
- removed R25: 100k, Resistor_SMD:R_0603_1608Metric, symbol Device:R_US
- removed R27: 100k, Resistor_SMD:R_0603_1608Metric, symbol UAM_symbols:R_US
- removed R28: 10k, Resistor_SMD:R_0603_1608Metric, symbol UAM_symbols:R_US
- removed U11: TLV75733PDYDR, Package_SON:WSON-6-1EP_2x2mm_P0.65mm_EP1x1.6mm, symbol UAM_symbols:TLV75733PDYDR
- added R20: 100k, Resistor_SMD:R_0603_1608Metric, symbol Device:R_US
- added R21: 2k, Resistor_SMD:R_0603_1608Metric, symbol Device:R_US
- added R23: 4k7, Resistor_SMD:R_0603_1608Metric, symbol Device:R_US
- added R25: 1k, Resistor_SMD:R_0603_1608Metric, symbol UAM_symbols:R_US
- added U14: TLV75733PDRVR, Package_SON:WSON-6-1EP_2x2mm_P0.65mm_EP1x1.6mm, symbol UAM_symbols:TLV75733PDYDR
- added U7: TPS22919, Package_TO_SOT_SMD:SOT-363_SC-70-6, symbol UAM_symbols:TPS22919
- added U8: BV1HB045EFJ-C, Package_SO:HTSOP-8-1EP_3.9x4.9mm_P1.27mm_EP2.4x3.2mm, symbol UAM_symbols:BV1HB045EFJ-C
- R22: value 100k -> 4k7; LCSC PN C25803 -> C23162
- U13: renamed from U10; value TLV75733PDYDR -> TLV75733PDRVR; LCSC PN C22399950 -> C2868428
- renumbered C26 to C23, C27 to C24, C23 to C26, C24 to C27, C29 to C28, C30 to C29, C31 to C30, C32 to C31, C33 to C32, C34 to C33, C35 to C34, C36 to C35, C37 to C36, C38 to C37, C39 to C38, C40 to C39, C41 to C40, C42 to C41, C43 to C42, C44 to C43, C45 to C44, C46 to C45, C47 to C46, C48 to C47, C49 to C48, C50 to C49, C51 to C50, C52 to C51, C53 to C52, C54 to C53, C55 to C54, C56 to C55, C57 to C56, C58 to C57, C59 to C58, C60 to C59, C61 to C60, C62 to C61, Q7 to Q2, R23 to R24, R29 to R27, R30 to R28, R31 to R29, R32 to R30, R33 to R31, R34 to R32, R35 to R33, R36 to R34, R37 to R35, R38 to R36, R39 to R37, R40 to R38, R41 to R39, U7 to U10, U8 to U11, U9 to U12, U12 to U15, U6 to U9
Connections:
- net +3.3VA: now also U14.1 (OUT)
- net +30V: now also D2.3; no longer D2.1
- net +30Va: now also D2.1; no longer D2.3
- net +5V: now also U14.6 (IN), U7.1 (IN); no longer R22.1
- net +BATT: now also U8.9 (VBB); no longer C26.1, C27.1, C29.1, L1.1, U11.1 (BIAS)
- net 3V3A_EN: now also U14.4 (EN)
- net GND: now also R20.1, R23.2, R25.2, U14.3 (GND), U14.7 (EPAD), U7.2 (GND), U8.1 (GND)
- net N5V_5V: now also U7.5 (QOD), U7.6 (OUT)
- net 5V_SWa: now reaches L2.1, U9.7 (SW)
- net 30V_EN: now reaches R22.2
- net 30V_BIAS: now reaches U11.12 (UVLO_SYNC)
- net 30V_BIAS: now also C26.1, C27.1, C29.1, L1.1, U11.1 (BIAS), U8.5 (OUT), U8.6 (OUT), U8.7 (OUT), U8.8 (OUT)
- net 26V_COMP renamed 30V_COMP
- net 26V_COMPa renamed 30V_COMPa
- new net: R25.1, U8.4 (SENSE)
- new net: R21.2, U7.3 (ON)
- new net: U14.2 (NC), U14.5 (NC)
- new net: R22.1, U8.2 (IN)
- new net: R23.1, U8.3 (SEN)
- new net -5V_EN: R20.2, R21.1
- no-connect marks 6 -> 7
Other:
- note added: "12V Buck Converter"
- note added: "Inductor msut be oversized in case of output short circuit. Could reduce component size requirements by chossing buck converter with lower max output current"
- note added: "Internally pulled down active high"
- moved on the sheet: C25, C26, C27, C29, C41, C42, C43, C44, C48, C50, C51, C52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
