File: v2/src/Feedback.kicad_sch (KiCad schematic)
At the start: 26 parts, among them Q16 BSS138, Q17 DMP3068L-7, Q18 BSS138, U20 OPA991SIDBVR, U21 TS5A4624, U22 OPA991SIDBVR

Commit message: v2.0 final version including minor hardware revisions
Parts:
- removed R101: 10k, Resistor_SMD:R_0603_1608Metric, symbol UAM_symbols:R_US
- added R117: 10k, Resistor_SMD:R_0603_1608Metric, symbol Device:R_US
- added R89: 100k, Resistor_SMD:R_0603_1608Metric, symbol UAM_symbols:R_US
- C111: renamed from C112; value 100n -> 10u; LCSC PN C14663 -> C2959727
- renumbered C108 to C107, C109 to C108, C110 to C109, C111 to C110, C113 to C112, C114 to C113, Q16 to Q10, Q17 to Q11, Q18 to Q12, R93 to R81, R94 to R82, R95 to R83, R96 to R84, R97 to R85, R98 to R86, R99 to R87, R100 to R88, R102 to R90, R103 to R91, R104 to R92, U20 to U23, U21 to U24, U22 to U25
Connections:
- net -3V3: now also R117.1
- net GND: now also R89.2
- net at C111.2, U25.3 (+): now also R89.1
- net IN_FB_EN# renamed IN_FB_EN
- net IN_FB_EN: now also R117.2
