File: v2/src/Impedance_matching.kicad_sch (KiCad schematic)
At the start: 12 parts

Commit message: v2.0 final version including minor hardware revisions
Parts:
- removed TP14, TP15: TestPoint, TestPoint:TestPoint_Pad_D1.0mm, symbol UAM_symbols:TestPoint
- renumbered C124 to C123, C125 to C124, C126 to C125, C127 to C126, C128 to C127
Changed lines of the file:
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@@
-	)
-	(junction
-		(at 162.56 67.31)
-		(diameter 0)
-		(color 0 0 0 0)
 	)
 	(junction
@@
 	)
 	(junction
-		(at 74.93 67.31)
-		(diameter 0)
-		(color 0 0 0 0)
-	)
-	(junction
 		(at 97.79 55.88)
 		(diameter 0)
@@
 	(wire
 		(pts
-			(xy 162.56 67.31) (xy 173.99 67.31)
-		)
-		(stroke
-			(width 0)
-			(type default)
-		)
-	)
-	(wire
-		(pts
 			(xy 109.22 67.31) (xy 119.38 67.31)
 		)
@@
 	(wire
 		(pts
-			(xy 148.59 67.31) (xy 162.56 67.31)
+			(xy 148.59 67.31) (xy 173.99 67.31)
 		)
 		(stroke
@@
 	)
 	(symbol
-		(lib_id "UAM_symbols:TestPoint")
-		(at 74.93 67.31 0)
-		(unit 1)
-		(exclude_from_sim no)
-		(in_bom yes)
-		(on_board yes)
-		(dnp no)
-		(fields_autoplaced yes)
-		(property "Reference" "TP14"
-			(at 77.47 62.7379 0)
-			(effects
-				(font
-					(size 1.27 1.27)
-				)
-				(justify left)
-			)
-		)
-		(property "Value" "TestPoint"
-			(at 77.47 65.2779 0)
-			(effects
-				(font
-					(size 1.27 1.27)
-				)
-				(justify left)
-			)
-		)
-		(property "Footprint" "TestPoint:TestPoint_Pad_D1.0mm"
-			(at 80.01 67.31 0)
-			(effects
-				(font
-					(size 1.27 1.27)
-				)
-				(hide yes)
-			)
-		)
-		(property "Datasheet" "~"
-			(at 80.01 67.31 0)
-			(effects
-				(font
-					(size 1.27 1.27)
-				)
-				(hide yes)
-			)
-		)
-		(property "Description" "test point"
-			(at 74.93 67.31 0)
-			(effects
-				(font
-					(size 1.27 1.27)
-				)
-				(hide yes)
-			)
-		)
-		(property "MPN" ""
-			(at 74.93 67.31 0)
-			(effects
-				(font
-					(size 1.27 1.27)
-				)
-			)
-		)
-		(pin "1"
-		)
-		(instances
-			(project "OpenAquatix-Hardware"
-				(path "/af15edda-fefd-41c1-b558-f4be36e6b138/890d2ccc-0ee1-44af-a69f-0d759033bbe5"
-					(reference "TP14")
-					(unit 1)
-				)
-			)
-		)
-	)
-	(symbol
 		(lib_id "UAM_symbols:SMAJ85CA")
 		(at 119.38 76.2 90)
@@
 		(dnp no)
 		(fields_autoplaced yes)
-		(property "Reference" "#PWR0199"
+		(property "Reference" "#PWR0202"
 			(at 116.84 92.71 0)
 			(effects
@@
 			(project "OpenAquatix-Hardware"
 				(path "/af15edda-fefd-41c1-b558-f4be36e6b138/890d2ccc-0ee1-44af-a69f-0d759033bbe5"
-					(reference "#PWR0199")
+					(reference "#PWR0202")
 					(unit 1)
 				)
@@
 		(exclude_from_sim no)
 		(in_bom no)
-		(on_board yes)
+		(on_board no)
 		(dnp yes)
-		(property "Reference" "C126"
+		(property "Reference" "C125"
 			(at 101.6 50.8 90)
 			(effects
@@
 				)
 				(hide yes)
+			)
+		)
+		(property "MPN" ""
+			(at 101.6 55.88 0)
+			(effects
+				(font
+					(size 1.27 1.27)
+				)
 			)
 		)
@@
 			(project "OpenAquatix-Hardware"
 				(path "/af15edda-fefd-41c1-b558-f4be36e6b138/890d2ccc-0ee1-44af-a69f-0d759033bbe5"
-					(reference "C126")
+					(reference "C125")
 					(unit 1)
 				)
@@
 		(exclude_from_sim no)
 		(in_bom no)
-		(on_board yes)
+		(on_board no)
 		(dnp yes)
 		(fields_autoplaced yes)
-		(property "Reference" "C127"
+		(property "Reference" "C126"
 			(at 101.6 59.69 90)
 			(effects
@@
 			(project "OpenAquatix-Hardware"
 				(path "/af15edda-fefd-41c1-b558-f4be36e6b138/890d2ccc-0ee1-44af-a69f-0d759033bbe5"
-					(reference "C127")
+					(reference "C126")
 					(unit 1)
 				)
@@
 		(exclude_from_sim no)
 		(in_bom no)
-		(on_board yes)
+		(on_board no)
 		(dnp yes)
-		(property "Reference" "C125"
+		(property "Reference" "C124"
 			(at 101.6 41.91 90)
 			(effects
@@
 				)
 				(hide yes)
+			)
+		)
+		(property "MPN" ""
+			(at 101.6 46.99 0)
+			(effects
+				(font
+					(size 1.27 1.27)
+				)
 			)
 		)
@@
 			(project "OpenAquatix-Hardware"
 				(path "/af15edda-fefd-41c1-b558-f4be36e6b138/890d2ccc-0ee1-44af-a69f-0d759033bbe5"
-					(reference "C125")
-					(unit 1)
-				)
-			)
-		)
-	)
-	(symbol
-		(lib_id "UAM_symbols:TestPoint")
-		(at 162.56 67.31 0)
-		(unit 1)
-		(exclude_from_sim no)
-		(in_bom yes)
-		(on_board yes)
-		(dnp no)
-		(fields_autoplaced yes)
-		(property "Reference" "TP15"
-			(at 165.1 62.7379 0)
-			(effects
-				(font
-					(size 1.27 1.27)
-				)
-				(justify left)
-			)
-		)
-		(property "Value" "TestPoint"
-			(at 165.1 65.2779 0)
-			(effects
-				(font
-					(size 1.27 1.27)
-				)
-				(justify left)
-			)
-		)
-		(property "Footprint" "TestPoint:TestPoint_Pad_D1.0mm"
-			(at 167.64 67.31 0)
-			(effects
-				(font
-					(size 1.27 1.27)
-				)
-				(hide yes)
-			)
-		)
-		(property "Datasheet" "~"
-			(at 167.64 67.31 0)
-			(effects
-				(font
-					(size 1.27 1.27)
-				)
-				(hide yes)
-			)
-		)
-		(property "Description" "test point"
-			(at 162.56 67.31 0)
-			(effects
-				(font
-					(size 1.27 1.27)
-				)
-				(hide yes)
-			)
-		)
-		(pin "1"
-		)
-		(instances
-			(project "OpenAquatix-Hardware"
-				(path "/af15edda-fefd-41c1-b558-f4be36e6b138/890d2ccc-0ee1-44af-a69f-0d759033bbe5"
-					(reference "TP15")
+					(reference "C124")
 					(unit 1)
 				)
@@
 		(dnp no)
 		(fields_autoplaced yes)
-		(property "Reference" "C124"
+		(property "Reference" "C123"
 			(at 101.6 30.48 90)
 			(effects
@@
 			(project "OpenAquatix-Hardware"
 				(path "/af15edda-fefd-41c1-b558-f4be36e6b138/890d2ccc-0ee1-44af-a69f-0d759033bbe5"
-					(reference "C124")
+					(reference "C123")
 					(unit 1)
 				)
@@
 		(dnp no)
 		(fields_autoplaced yes)
-		(property "Reference" "#PWR0200"
+		(property "Reference" "#PWR0203"
 			(at 148.59 96.52 0)
 			(effects
@@
 			(project "OpenAquatix-Hardware"
 				(path "/af15edda-fefd-41c1-b558-f4be36e6b138/890d2ccc-0ee1-44af-a69f-0d759033bbe5"
-					(reference "#PWR0200")
+					(reference "#PWR0203")
 					(unit 1)
 				)
@@
 		(exclude_from_sim no)
 		(in_bom no)
-		(on_board yes)
+		(on_board no)
 		(dnp yes)
 		(fields_autoplaced yes)
-		(property "Reference" "C128"
+		(property "Reference" "C127"
 			(at 113.03 74.9299 0)
 			(effects
@@
 				)
 				(hide yes)
+			)
+		)
+		(property "MPN" ""
+			(at 109.22 76.2 0)
+			(effects
+				(font
+					(size 1.27 1.27)
+				)
 			)
 		)
@@
 			(project "OpenAquatix-Hardware"
 				(path "/af15edda-fefd-41c1-b558-f4be36e6b138/890d2ccc-0ee1-44af-a69f-0d759033bbe5"
-					(reference "C128")
+					(reference "C127")
 					(unit 1)
 				)
