File: v2/src/STM32.kicad_sch (KiCad schematic)
At the start: 67 parts, among them J1 Conn_ARM_JTAG_SWD_10, J2 USB_B_Micro, Q1 BSS138, Q2 DMP3068L-7, Q3 BSS138, SW1 SW_Push, SW2 SW_Push, U1 W25Q16JVSS, U2 STM32H723VET6, U3 TS5A4624, U4 TPD4E05U06DQA, U5 TPD4E05U06DQA, Y1 32.768 kHz, Y2 8 MHz

Commit message: v2.0 final version including minor hardware revisions
Parts:
- removed Q2: DMP3068L-7, Package_TO_SOT_SMD:SOT-23, symbol Transistor_FET:DMP3099L
- removed Q3: BSS138, Package_TO_SOT_SMD:SOT-23, symbol UAM_symbols:BSS138
- removed R20: 2k, Resistor_SMD:R_0603_1608Metric, symbol Device:R_US
- removed R21: 100k, Resistor_SMD:R_0603_1608Metric, symbol Device:R_US
- removed R9: 22R, Resistor_SMD:R_0603_1608Metric, symbol Device:R_US
- removed TP10, TP5, TP6, TP7, TP8, TP9: TestPoint_Small, TestPoint:TestPoint_Pad_D1.0mm, symbol UAM_symbols:TestPoint_Small
- removed TP3, TP4: TestPoint, TestPoint:TestPoint_Pad_D1.0mm, symbol UAM_symbols:TestPoint
- added R18: 100k, Resistor_SMD:R_0603_1608Metric, symbol Device:R_US
- added U6: TPS22919, Package_TO_SOT_SMD:SOT-363_SC-70-6, symbol UAM_symbols:TPS22919
- J1: FT Rotation Offset (none) -> 90
- R19: value 100k -> 2k; LCSC PN C25803 -> C22975
- Y1: footprint OpenAquatix-Hardware_footprints:MP06734 -> Crystal:Crystal_SMD_3225-4Pin_3.2x2.5mm; LCSC PN (none) -> C213398; MPN MP06734 -> 1XZA032768AD19
- renumbered R11 to R10, R12 to R11, R13 to R12, R14 to R13, R16 to R14, R17 to R16, R18 to R17, R10 to R9
Connections:
- net +5V: now also U6.1 (IN); no longer R19.1
- net GND: now also R18.1, U6.2 (GND)
- net INPUT_FB_EN: now also U2.54 (PB15); no longer U2.53 (PB14)
- net OUTPUT_FB_EN#: now also U2.53 (PB14); no longer U2.54 (PB15)
- net PAMP_FILTER_EN#: now also U2.45 (PE15); no longer U2.43 (PE13)
- net RESET#: no longer U4.5 (D2-), U4.6 (NC)
- net SWO: now also U4.5 (D2-), U4.6 (NC); no longer U4.4 (D2+), U4.7 (NC)
- net TPA_RESET: now also U2.43 (PE13); no longer U2.23 (PA1), U2.45 (PE15)
- net ULPI_STP: now also U2.15 (PC0)
- net WS_5V: now also U6.5 (QOD), U6.6 (OUT)
- net WS_EN: now also R19.1, R18.2
- net at R19.2: now also U6.3 (ON)
- net -5V_EN# renamed -5V_EN
- net 30V_EN# renamed 30V_EN
- no-connect marks 13 -> 16
Other:
- note added: "Note: LSE has potentially high start time of 3s Could be an issue when first booting"
- moved on the sheet: TP2
