File: v2/src/TR_Switch.kicad_sch (KiCad schematic)
At the start: 8 parts, among them K1 3570.1419.051, Q19 BSS138, U31 TS5A4624, U32 AQY210S

Commit message: v2.0 final version including minor hardware revisions
Parts:
- renumbered C148 to C147, Q19 to Q13, R125 to R113, R126 to R114, U31 to U34, U32 to U35
Other:
- note added: "Doubles as current setting resistor for PhotoMOS and gate resistor for reed relay"
- note removed: "R126 doubles as current setting resistor for PhotoMOS and gate resistor for reed relay"
Changed lines of the file:
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@@
 		(rev "2.0")
 	)
-	(text "R126 doubles as current setting resistor for PhotoMOS\nand gate resistor for reed relay"
+	(text "Doubles as current setting resistor for PhotoMOS\nand gate resistor for reed relay"
 		(exclude_from_sim no)
 		(at 80.264 93.472 0)
@@
 		(dnp no)
 		(fields_autoplaced yes)
-		(property "Reference" "U31"
+		(property "Reference" "U34"
 			(at 57.15 73.66 0)
 			(effects
@@
 			(project "OpenAquatix-Hardware"
 				(path "/af15edda-fefd-41c1-b558-f4be36e6b138/fb9c5bf4-ce8e-4e79-bb83-62ffc4865bf7"
-					(reference "U31")
+					(reference "U34")
 					(unit 1)
 				)
@@
 		(on_board yes)
 		(dnp no)
-		(property "Reference" "Q19"
+		(property "Reference" "Q13"
 			(at 171.45 88.8999 0)
 			(effects
@@
 			(project "OpenAquatix-Hardware"
 				(path "/af15edda-fefd-41c1-b558-f4be36e6b138/fb9c5bf4-ce8e-4e79-bb83-62ffc4865bf7"
-					(reference "Q19")
+					(reference "Q13")
 					(unit 1)
 				)
@@
 		(dnp no)
 		(fields_autoplaced yes)
-		(property "Reference" "#PWR0240"
+		(property "Reference" "#PWR0243"
 			(at 40.64 101.6 0)
 			(effects
@@
 			(project ""
 				(path "/af15edda-fefd-41c1-b558-f4be36e6b138/fb9c5bf4-ce8e-4e79-bb83-62ffc4865bf7"
-					(reference "#PWR0240")
+					(reference "#PWR0243")
 					(unit 1)
 				)
@@
 		(dnp no)
 		(fields_autoplaced yes)
-		(property "Reference" "#PWR0241"
+		(property "Reference" "#PWR0244"
 			(at 143.51 41.91 0)
 			(effects
@@
 			(project "OpenAquatix-Hardware"
 				(path "/af15edda-fefd-41c1-b558-f4be36e6b138/fb9c5bf4-ce8e-4e79-bb83-62ffc4865bf7"
-					(reference "#PWR0241")
+					(reference "#PWR0244")
 					(unit 1)
 				)
@@
 		(on_board yes)
 		(dnp no)
-		(property "Reference" "R125"
+		(property "Reference" "R113"
 			(at 27.686 84.582 0)
 			(effects
@@
 			(project "OpenAquatix-Hardware"
 				(path "/af15edda-fefd-41c1-b558-f4be36e6b138/fb9c5bf4-ce8e-4e79-bb83-62ffc4865bf7"
-					(reference "R125")
+					(reference "R113")
 					(unit 1)
 				)
@@
 		(dnp no)
 		(fields_autoplaced yes)
-		(property "Reference" "#PWR0238"
+		(property "Reference" "#PWR0241"
 			(at 30.48 95.25 0)
 			(effects
@@
 			(project "OpenAquatix-Hardware"
 				(path "/af15edda-fefd-41c1-b558-f4be36e6b138/fb9c5bf4-ce8e-4e79-bb83-62ffc4865bf7"
-					(reference "#PWR0238")
+					(reference "#PWR0241")
 					(unit 1)
 				)
@@
 		(on_board yes)
 		(dnp no)
-		(property "Reference" "C148"
+		(property "Reference" "C147"
 			(at 43.434 90.17 0)
 			(effects
@@
 			(project ""
 				(path "/af15edda-fefd-41c1-b558-f4be36e6b138/fb9c5bf4-ce8e-4e79-bb83-62ffc4865bf7"
-					(reference "C148")
+					(reference "C147")
 					(unit 1)
 				)
@@
 		(dnp no)
 		(fields_autoplaced yes)
-		(property "Reference" "#PWR0242"
+		(property "Reference" "#PWR0245"
 			(at 160.02 74.93 0)
 			(effects
@@
 			(project ""
 				(path "/af15edda-fefd-41c1-b558-f4be36e6b138/fb9c5bf4-ce8e-4e79-bb83-62ffc4865bf7"
-					(reference "#PWR0242")
+					(reference "#PWR0245")
 					(unit 1)
 				)
@@
 		(on_board yes)
 		(dnp no)
-		(property "Reference" "#PWR0239"
+		(property "Reference" "#PWR0242"
 			(at 40.64 91.44 0)
 			(effects
@@
 			(project ""
 				(path "/af15edda-fefd-41c1-b558-f4be36e6b138/fb9c5bf4-ce8e-4e79-bb83-62ffc4865bf7"
-					(reference "#PWR0239")
+					(reference "#PWR0242")
 					(unit 1)
 				)
@@
 		(dnp no)
 		(fields_autoplaced yes)
-		(property "Reference" "#PWR0243"
+		(property "Reference" "#PWR0246"
 			(at 167.64 101.6 0)
 			(effects
@@
 			(project "OpenAquatix-Hardware"
 				(path "/af15edda-fefd-41c1-b558-f4be36e6b138/fb9c5bf4-ce8e-4e79-bb83-62ffc4865bf7"
-					(reference "#PWR0243")
+					(reference "#PWR0246")
 					(unit 1)
 				)
@@
 		(dnp no)
 		(fields_autoplaced yes)
-		(property "Reference" "U32"
+		(property "Reference" "U35"
 			(at 156.21 22.86 0)
 			(effects
@@
 		(instances
 			(project ""
+				(path "/af15edda-fefd-41c1-b558-f4be36e6b138/0766ad09-d624-4487-92bd-10697a6e5161"
+					(reference "U32")
+					(unit 1)
+				)
 				(path "/af15edda-fefd-41c1-b558-f4be36e6b138/fb9c5bf4-ce8e-4e79-bb83-62ffc4865bf7"
-					(reference "U32")
+					(reference "U35")
 					(unit 1)
 				)
@@
 		(on_board yes)
 		(dnp no)
-		(property "Reference" "R126"
+		(property "Reference" "R114"
 			(at 73.66 85.598 90)
 			(effects
@@
 			(project "OpenAquatix-Hardware"
 				(path "/af15edda-fefd-41c1-b558-f4be36e6b138/fb9c5bf4-ce8e-4e79-bb83-62ffc4865bf7"
-					(reference "R126")
+					(reference "R114")
 					(unit 1)
 				)
