File: v2/src/pre_amplifier.kicad_sch (KiCad schematic)
At the start: 22 parts, among them U23 LM6211, U24 LMV641MFX/NOPB

Commit message: v2.0 final version including minor hardware revisions
Parts:
- removed TP11, TP12, TP13: TestPoint, TestPoint:TestPoint_Pad_D1.0mm, symbol UAM_symbols:TestPoint
- U26: renamed from U23; footprint Package_TO_SOT_SMD:TSOT-23-5 -> Package_TO_SOT_SMD:SOT-23-5
- renumbered C116 to C114, C117 to C115, C118 to C116, C119 to C117, C115 to C118, C120 to C119, C121 to C120, C122 to C121, C123 to C122, R112 to R100, R105 to R93, R106 to R94, R107 to R95, R108 to R96, R109 to R97, R110 to R98, R111 to R99, U24 to U27
Connections:
- net PREAMP_LPF renamed PREAMP_BPF
